Commit message: updated

File: two_links_robot_description/two_links_robot_description.urdf (robot description, URDF)
Before this commit: robot two_DOF_robot, 4 links, 3 joints
Joints:
- joint joint2: origin xyz=0 0 2 rpy=0 0 0 -> xyz=0 0 1 rpy=0 0 0

Commit message: not fixed yet

File: two_links_robot_description/two_links_robot_description.urdf (robot description, URDF)
Before this commit: robot two_DOF_robot, 4 links, 3 joints
Links:
- removed link link2
Joints:
- removed joint joint2

Commit message: joints_trajectory_action_server.cpp and joints_trajectory_action_client.cpp files have been debugged.

File: two_links_robot_description/two_links_robot_description.urdf (robot description, URDF)
Before this commit: robot two_DOF_robot, 3 links, 2 joints
Links:
- added link link2, mass 1; collision cylinder length=1 radius=0.1; visual cylinder length=1 radius=0.1
Joints:
- added joint joint2: type continuous, parent link1, child link2, origin xyz=0 0 1 rpy=0 0 0, axis 0 1 0
